Commit message: tmp commit

File: open_manipulator_description/urdf/open_manipulator.gazebo.xacro (robot description, xacro)
@@ -24,14 +24,6 @@
   <!-- Link4 -->
   <RefLink ref="link4"/>
-  <!-- Link5 -->
-  <RefLink ref="link5"/>
   <!-- gripper_link -->
   <RefLink ref="gripper_link"/>
-  <!-- gripper_link_sub -->
-  <RefLink ref="gripper_link_sub"/>
-  <!-- end effector link -->
-  <gazebo reference="end_effector_link">
-    <material>Gazebo/Red</material>
-  </gazebo>
   <!-- ros_control plugin -->
   <gazebo>

File: open_manipulator_description/urdf/open_manipulator.urdf.xacro (robot description, xacro)
@@ -178,59 +178,6 @@
     </inertial>
   </link>
-  <!--  Joint 4 -->
-  <joint name="joint4" type="revolute">
-    <parent link="link4"/>
-    <child link="link5"/>
-    <origin xyz="0.124 0.0 0.0" rpy="0 0 0"/>
-    <axis xyz="0 1 0"/>
-    <limit velocity="4.8" effort="1" lower="${-pi*0.57}" upper="${pi*0.65}" />
-  </joint>
-  <!-- Transmission 4 -->
-  <xacro:SimpleTransmission n="4" joint="joint4" />
-  <!--  Link 5 -->
-  <link name="link5">
-    <visual>
-      <origin xyz="0 0 0" rpy="0 0 0"/>
-      <geometry>
-        <mesh filename="package://open_manipulator_description/meshes/chain_link5.stl" scale="0.001 0.001 0.001"/>
-      </geometry>
-      <material name="grey"/>
-    </visual>
-    <collision>
-      <origin xyz="0 0 0" rpy="0 0 0"/>
-      <geometry>
-        <mesh filename="package://open_manipulator_description/meshes/chain_link5.stl" scale="0.001 0.001 0.001"/>
-      </geometry>
-    </collision>
-<!--    <inertial>
-      <origin xyz="0 0 0" />
-      <mass value="0.141" />
-      <inertia ixx="0.1" ixy="0.0" ixz="0.0"
-               iyy="0.1" iyz="0.0"
-               izz="0.1" />
-    </inertial>-->
-     <inertial>
-      <origin xyz="4.4206755e-02 3.6839985e-07 8.9142216e-03" />
-      <mass value="1.4327573e-01" />
-      <inertia ixx="8.0870749e-05" ixy="0.0" ixz="-1.0157896e-06"
-               iyy="7.5980465e-05" iyz="0.0"
-               izz="9.3127351e-05" />
-    </inertial>
-  </link>
   <!--  Gripper link -->
   <link name="gripper_link">
-    <visual>
-      <origin xyz="0.0 0.0 0" rpy="0 0 0"/>
-      <geometry>
-        <mesh filename="package://open_manipulator_description/meshes/chain_link_grip_l.stl" scale="0.001 0.001 0.001"/>
-      </geometry>
-      <material name="grey"/>
-    </visual>
-    <collision>
-      <origin xyz="0.0 0.0 0" rpy="0 0 0"/>
-      <geometry>
-        <mesh filename="package://open_manipulator_description/meshes/chain_link_grip_l.stl" scale="0.001 0.001 0.001"/>
-      </geometry>
-    </collision>
     <inertial>
       <origin xyz="0 0 0" />
@@ -240,15 +187,8 @@
                izz="1.0e-03" />
     </inertial>
-<!--     <inertial>
-      <origin xyz="${0.028 + 8.3720668e-03} ${0.0246 + 9.9696160e-03} -4.2836895e-07" />
-      <mass value="3.2218127e-02" />
-      <inertia ixx="9.5568826e-06" ixy="2.8424644e-06" ixz="-3.2829197e-10"
-               iyy="2.2552871e-05" iyz="-3.1463634e-10"
-               izz="1.7605306e-05" />
-    </inertial>-->
   </link>
   <!--  Gripper joint -->
   <joint name="gripper" type="prismatic">
-    <parent link="link5"/>
+    <parent link="link4"/>
     <child link="gripper_link"/>
     <origin xyz="0.0817 0.021 0.0" rpy="0 0 0"/>
@@ -258,65 +198,3 @@
   <!-- Transmission 5 -->
   <xacro:SimpleTransmission n="5" joint="gripper" />
-  <!--  Gripper link sub -->
-  <link name="gripper_link_sub">
-    <visual>
-      <origin xyz="0.0 -0.0 0" rpy="0 0 0"/>
-      <geometry>
-        <mesh filename="package://open_manipulator_description/meshes/chain_link_grip_r.stl" scale="0.001 0.001 0.001"/>
-      </geometry>
-      <material name="grey"/>
-    </visual>
-    <collision>
-      <origin xyz="0.0 -0.0 0" rpy="0 0 0"/>
-      <geometry>
-        <mesh filename="package://open_manipulator_description/meshes/chain_link_grip_r.stl" scale="0.001 0.001 0.001"/>
-      </geometry>
-    </collision>
-    <inertial>
-      <origin xyz="0 0 0" />
-      <mass value="0.017" />
-      <inertia ixx="1.0e-03" ixy="0.0" ixz="0.0"
-               iyy="1.0e-03" iyz="0.0"
-               izz="1.0e-03" />
-    </inertial>
-<!--     <inertial>
-      <origin xyz="${0.028 + 8.3720668e-03} ${-0.0246 - 9.9696160e-03} -4.2836895e-07" />
-      <mass value="3.2218127e-02" />
-      <inertia ixx="9.5568826e-06" ixy="2.8424644e-06" ixz="-3.2829197e-10"
-               iyy="2.2552871e-05" iyz="-3.1463634e-10"
-               izz="1.7605306e-05" />
-    </inertial>-->
-  </link>
-  <!--  Gripper joint sub -->
-  <joint name="gripper_sub" type="prismatic">
-    <parent link="link5"/>
-    <child link="gripper_link_sub"/>
-    <origin xyz="0.0817 -0.021 0" rpy="0 0 0"/>
-    <axis xyz="0 -1 0"/>
-    <limit velocity="4.8" effort="1" lower="-0.010" upper="0.019" />
-    <mimic joint="gripper" multiplier="1"/>
-  </joint>
-  <!-- Transmission 6 -->
-  <xacro:SimpleTransmission n="6" joint="gripper_sub" />
-  <!-- end effector joint -->
-  <joint name="end_effector_joint" type="fixed">
-    <origin xyz="0.126 0.0 0.0" rpy="0 0 0"/>
-    <parent link="link5"/>
-    <child link="end_effector_link"/>
-  </joint>
-  <!-- end effector link -->
-  <link name="end_effector_link">
-    <visual>
-      <origin xyz="0 0 0" rpy="0 0 0"/>
-      <geometry>
-        <box size="0.01 0.01 0.01" />
-      </geometry>
-      <material name="red"/>
-     </visual>
-    <inertial>
-      <origin xyz="0.0 0.0 0.0" rpy="0 0 0"/>
-      <mass value="0.001"/>
-      <inertia ixx="1.0e-06" ixy="0.0" ixz="0.0" iyy="1.0e-06" iyz="0.0" izz="1.0e-06" />
-    </inertial>
-  </link>
 </robot>

Commit message: Removing gripper changes

File: open_manipulator_description/urdf/open_manipulator.gazebo.xacro (robot description, xacro)
@@ -1,38 +1,40 @@
 <?xml version="1.0"?>
-<robot xmlns:xacro="http://ros.org/wiki/xacro">
-  <!-- Gazebo Reference macro -->
-  <xacro:macro name="RefLink" params="ref">
-    <gazebo reference="${ref}">
-      <kp>1000000.0</kp>
-      <kd>100.0</kd>
-      <mu1>30.0</mu1>
-      <mu2>30.0</mu2>
-      <maxVel>1.0</maxVel>
-      <minDepth>0.001</minDepth>
-      <material>Gazebo/DarkGrey</material>
-    </gazebo>
-  </xacro:macro>
-  <!-- World -->
-  <gazebo reference="world"/>
-  <!-- Link1 -->
-  <RefLink ref="link1"/>
-  <!-- Link2 -->
-  <RefLink ref="link2"/>
-  <!-- Link3 -->
-  <RefLink ref="link3"/>
-  <!-- Link4 -->
-  <RefLink ref="link4"/>
-  <!-- Link5 -->
-  <RefLink ref="link5"/>
+<robot
+	xmlns:xacro="http://ros.org/wiki/xacro">
+	<!-- Gazebo Reference macro -->
+	<xacro:macro name="RefLink" params="ref">
+		<gazebo reference="${ref}">
+			<kp>1000000.0</kp>
+			<kd>100.0</kd>
+			<mu1>30.0</mu1>
+			<mu2>30.0</mu2>
+			<maxVel>1.0</maxVel>
+			<minDepth>0.001</minDepth>
+			<material>Gazebo/DarkGrey</material>
+		</gazebo>
+	</xacro:macro>
+	<!-- World -->
+	<gazebo reference="world"/>
+	<!-- Link1 -->
+	<RefLink ref="link1"/>
+	<!-- Link2 -->
+	<RefLink ref="link2"/>
+	<!-- Link3 -->
+	<RefLink ref="link3"/>
+	<!-- Link4 -->
+	<RefLink ref="link4"/>
+	<!-- Link5 -->
+	<RefLink ref="link5"/>
+</robot>
   <!-- gripper_link -->
-  <RefLink ref="gripper_link"/>
+  <!-- <RefLink ref="gripper_link"/> -->
   <!-- gripper_link_sub -->
-  <RefLink ref="gripper_link_sub"/>
+  <!-- <RefLink ref="gripper_link_sub"/> -->
   <!-- end effector link -->
-  <gazebo reference="end_effector_link">
+  <!-- <gazebo reference="end_effector_link">
     <material>Gazebo/Red</material>
-  </gazebo>
+  </gazebo> -->
   <!-- ros_control plugin -->
-  <gazebo>
+  <!-- <gazebo>
     <plugin name="gazebo_ros_control" filename="libgazebo_ros_control.so">
       <controlPeriod>0.001</controlPeriod>
@@ -40,8 +42,8 @@
       <legacyModeNS>true</legacyModeNS>
     </plugin>
-  </gazebo>
-  <gazebo>
+  </gazebo> -->
+  <!-- <gazebo> -->
     <!-- loading plugin: mimic joints works in gazebo now -->
-    <plugin name="gazebo_gripper_ros_control" filename="libroboticsgroup_gazebo_mimic_joint_plugin.so">
+    <!-- <plugin name="gazebo_gripper_ros_control" filename="libroboticsgroup_gazebo_mimic_joint_plugin.so">
       <joint>gripper</joint>
       <mimicJoint>gripper_sub</mimicJoint>
@@ -49,7 +51,7 @@
       <offset>0.0</offset>
     </plugin>
-  </gazebo>
+  </gazebo> -->
   <!-- camera -->
-  <gazebo reference="camera_link">
+  <!-- <gazebo reference="camera_link">
     <sensor type="camera" name="intel_realsense_r200">
       <update_rate>30.0</update_rate>
@@ -66,9 +68,9 @@
         </clip>
         <noise>
-          <type>gaussian</type>
+          <type>gaussian</type> -->
           <!-- Noise is sampled independently per pixel on each frame.
                That pixel's noise value is added to each of its color
                channels, which at that point lie in the range [0,1]. -->
-          <mean>0.0</mean>
+          <!-- <mean>0.0</mean>
           <stddev>0.007</stddev>
         </noise>
@@ -89,4 +91,3 @@
       </plugin>
     </sensor>
-  </gazebo>
-</robot>
+  </gazebo> -->

File: open_manipulator_description/urdf/open_manipulator.transmission.xacro (robot description, xacro)
@@ -34,6 +34,6 @@
   <xacro:SimpleTransmissionPosition n="4" joint="joint4" />
   <!-- Transmission 5 -->
-  <xacro:SimpleTransmissionEffort n="5" joint="gripper" />
+  <!-- <xacro:SimpleTransmissionEffort n="5" joint="gripper" /> -->
   <!-- Transmission 6 -->
-  <xacro:SimpleTransmissionEffort n="6" joint="gripper_sub" />
+  <!-- <xacro:SimpleTransmissionEffort n="6" joint="gripper_sub" /> -->
 </robot>

File: open_manipulator_description/urdf/open_manipulator.urdf.xacro (robot description, xacro)
@@ -129,26 +129,29 @@
   <link name="link5">
     <visual>
-      <origin xyz="0 0 0" rpy="0 0 0"/>
+      <!-- <origin xyz="0 0 0" rpy="0 0 0"/>
       <geometry>
         <mesh filename="package://open_manipulator_description/meshes/chain_link5.stl" scale="0.001 0.001 0.001"/>
       </geometry>
-      <material name="grey"/>
-    </visual>
-    <collision>
-      <origin xyz="0 0 0" rpy="0 0 0"/>
+      <material name="grey"/> -->
+    ...
+    </visual>
+    <collision>
+      <!-- <origin xyz="0 0 0" rpy="0 0 0"/>
       <geometry>
         <mesh filename="package://open_manipulator_description/meshes/chain_link5.stl" scale="0.001 0.001 0.001"/>
-      </geometry>
-    </collision>
-    <inertial>
-      <origin xyz="4.4206755e-02 3.6839985e-07 8.9142216e-03" />
+      </geometry> -->
+    ...
+    </collision>
+    <inertial>
+      <!-- <origin xyz="4.4206755e-02 3.6839985e-07 8.9142216e-03" />
       <mass value="1.4327573e-01" />
       <inertia ixx="8.0870749e-05" ixy="0.0" ixz="-1.0157896e-06"
                iyy="7.5980465e-05" iyz="0.0"
-               izz="9.3127351e-05" />
+               izz="9.3127351e-05" /> -->
+    ...
     </inertial>
   </link>
   <!--  Gripper joint -->
-  <joint name="gripper" type="prismatic">
+  <!-- <joint name="gripper" type="prismatic">
     <parent link="link5"/>
     <child link="gripper_link"/>
@@ -156,7 +159,7 @@
     <axis xyz="0 1 0"/>
     <limit velocity="4.8" effort="1" lower="-0.010" upper="0.019" />
-  </joint>
+  </joint> -->
   <!--  Gripper link -->
-  <link name="gripper_link">
+  <!-- <link name="gripper_link">
     <visual>
       <origin xyz="0.0 0.0 0" rpy="0 0 0"/>
@@ -179,7 +182,7 @@
                izz="1.0e-03" />
     </inertial>
-  </link>
+  </link> -->
   <!--  Gripper joint sub -->
-  <joint name="gripper_sub" type="prismatic">
+  <!-- <joint name="gripper_sub" type="prismatic">
     <parent link="link5"/>
     <child link="gripper_link_sub"/>
@@ -188,7 +191,7 @@
     <limit velocity="4.8" effort="1" lower="-0.010" upper="0.019" />
     <mimic joint="gripper" multiplier="1"/>
-  </joint>
+  </joint> -->
   <!--  Gripper link sub -->
-  <link name="gripper_link_sub">
+  <!-- <link name="gripper_link_sub">
     <visual>
       <origin xyz="0.0 -0.0 0" rpy="0 0 0"/>
@@ -211,13 +214,13 @@
                izz="1.0e-03" />
     </inertial>
-  </link>
+  </link> -->
   <!-- end effector joint -->
-  <joint name="end_effector_joint" type="fixed">
+  <!-- <joint name="end_effector_joint" type="fixed">
     <origin xyz="0.126 0.0 0.0" rpy="0 0 0"/>
     <parent link="link5"/>
     <child link="end_effector_link"/>
-  </joint>
+  </joint> -->
   <!-- end effector link -->
-  <link name="end_effector_link">
+  <!-- <link name="end_effector_link">
     <visual>
       <origin xyz="0 0 0" rpy="0 0 0"/>
@@ -234,5 +237,5 @@
                izz="1.0e-03" />
     </inertial>
-  </link>
+  </link> -->
   <!-- Realsense Camera Joint Position -->
 <!--   <joint name="camera_joint" type="fixed">

Commit message: 4 joints no gripper

File: open_manipulator_description/urdf/open_manipulator.gazebo.xacro (robot description, xacro)
@@ -26,5 +26,4 @@
 	<!-- Link5 -->
 	<RefLink ref="link5"/>
-</robot>
   <!-- gripper_link -->
   <!-- <RefLink ref="gripper_link"/> -->
@@ -36,5 +35,5 @@
   </gazebo> -->
   <!-- ros_control plugin -->
-  <!-- <gazebo>
+  <gazebo>
     <plugin name="gazebo_ros_control" filename="libgazebo_ros_control.so">
       <controlPeriod>0.001</controlPeriod>
@@ -42,5 +41,5 @@
       <legacyModeNS>true</legacyModeNS>
     </plugin>
-  </gazebo> -->
+  </gazebo>
   <!-- <gazebo> -->
     <!-- loading plugin: mimic joints works in gazebo now -->
@@ -52,4 +51,5 @@
     </plugin>
   </gazebo> -->
+</robot>
   <!-- camera -->
   <!-- <gazebo reference="camera_link">

File: open_manipulator_description/urdf/open_manipulator.transmission.xacro (robot description, xacro)
@@ -32,7 +32,7 @@
   <xacro:SimpleTransmissionPosition n="3" joint="joint3" />
   <!-- Transmission 4 -->
-  <xacro:SimpleTransmissionPosition n="4" joint="joint4" />
+  <!-- <xacro:SimpleTransmissionPosition n="4" joint="joint4" /> -->
   <!-- Transmission 5 -->
-  <!-- <xacro:SimpleTransmissionEffort n="5" joint="gripper" /> -->
+  <xacro:SimpleTransmissionEffort n="5" joint="gripper" />
   <!-- Transmission 6 -->
   <!-- <xacro:SimpleTransmissionEffort n="6" joint="gripper_sub" /> -->

File: open_manipulator_description/urdf/open_manipulator.urdf.xacro (robot description, xacro)
@@ -119,5 +119,6 @@
   </link>
   <!--  Joint 4 -->
-  <joint name="joint4" type="revolute">
+  <!-- <joint name="joint4" type="revolute"> -->
+  <joint name="gripper" type="revolute">
     <parent link="link4"/>
     <child link="link5"/>
@@ -126,27 +127,29 @@
     <limit velocity="4.8" effort="1" lower="${-pi*0.57}" upper="${pi*0.65}" />
   </joint>
-  <!--  Link 5 -->
+   <!-- Link 5 fr12-h104 -->
   <link name="link5">
     <visual>
-      <!-- <origin xyz="0 0 0" rpy="0 0 0"/>
-      <geometry>
-        <mesh filename="package://open_manipulator_description/meshes/chain_link5.stl" scale="0.001 0.001 0.001"/>
-      </geometry>
-      <material name="grey"/> -->
+      <origin xyz="0 0 0" rpy="0 0 -1.57"/>
+      <geometry>
+        <!-- <mesh filename="package://open_manipulator_description/meshes/chain_link5.stl" scale="0.001 0.001 0.001"/>  -->
+        <mesh filename="package://open_manipulator_description/meshes/fr12-h104.stl" scale="0.001 0.001 0.001"/>
+      </geometry>
+      <material name="grey"/>
     ...
     </visual>
     <collision>
-      <!-- <origin xyz="0 0 0" rpy="0 0 0"/>
-      <geometry>
-        <mesh filename="package://open_manipulator_description/meshes/chain_link5.stl" scale="0.001 0.001 0.001"/>
-      </geometry> -->
+      <origin xyz="0 0 0" rpy="0 0 -1.57"/>
+      <geometry>
+        <!-- <mesh filename="package://open_manipulator_description/meshes/chain_link5.stl" scale="0.001 0.001 0.001"/> -->
+        <mesh filename="package://open_manipulator_description/meshes/fr12-h104.stl" scale="0.001 0.001 0.001"/>
+      </geometry>
     ...
     </collision>
     <inertial>
-      <!-- <origin xyz="4.4206755e-02 3.6839985e-07 8.9142216e-03" />
+      <origin xyz="4.4206755e-02 3.6839985e-07 8.9142216e-03" />
       <mass value="1.4327573e-01" />
       <inertia ixx="8.0870749e-05" ixy="0.0" ixz="-1.0157896e-06"
                iyy="7.5980465e-05" iyz="0.0"
-               izz="9.3127351e-05" /> -->
+               izz="9.3127351e-05" />
     ...
     </inertial>
